File: amp.kicad_pcb (KiCad board)
At the start: 2 copper layers, 11 parts, among them P2 CONN_01X02, P3 CONN_01X02, U1 TDA7385

Commit message: step2
Parts:
- added P4: CONN_01X02, Connectors:bornier2, F.Cu at (154.9, 123.2)
- added P5: CONN_01X02, Connectors:bornier2, F.Cu at (142.2, 123.2)
- added P6: CONN_01X02, Connectors:bornier2, F.Cu at (167.6, 123.2)
- added P7: CONN_01X02, Connectors:bornier2, F.Cu at (180.3, 123.2)
- moved C6 50.2 mm to (186.9, 103.6), turned to 270 degrees
- moved C5 40.7 mm to (133.1, 101.1), turned to 270 degrees
- moved P2 34.7 mm to (137.9, 70.6)
- moved C1 32.8 mm to (176.5, 108.6)
- moved C3 32.3 mm to (144.3, 108.6)
- moved C8 27.8 mm to (140.5, 102.4), turned to 180 degrees
- moved C7 12.3 mm to (180.6, 103.6)
- moved C4 4.37 mm to (158.5, 114.2)
- moved C2 1.35 mm to (162.6, 109.2)
Routing:
- net Net-(P5-Pad2): track 0.00 -> 25.2 mm
- net Net-(P5-Pad1): track 0.00 -> 23.9 mm
- net Net-(P7-Pad1): track 0.00 -> 23.1 mm
- net Net-(C6-Pad1): track 0.00 -> 23.1 mm
- net Net-(C5-Pad1): track 0.00 -> 21.4 mm
- net Net-(P6-Pad1): track 0.00 -> 21.2 mm
- net Net-(P6-Pad2): track 0.00 -> 20.8 mm
- net Net-(C7-Pad1): track 0.00 -> 20.5 mm
- net Net-(P4-Pad2): track 0.00 -> 20.1 mm
- net Net-(C8-Pad1): track 0.00 -> 19.3 mm
- net Net-(P4-Pad1): track 0.00 -> 18.8 mm
- net Net-(C3-Pad2): track 0.00 -> 17.3 mm
- net Net-(C1-Pad2): track 0.00 -> 17.1 mm
- net Net-(C2-Pad1): track 0.00 -> 4.24 mm
- net Net-(C4-Pad2): track 0.00 -> 4.22 mm

Commit message: final pcb for amp board
Parts:
- removed P2, P3, P4, P5, P6, P7: CONN_01X02, Connectors:bornier2
- added J10: CONN_01X01, PINTST, F.Cu at (172.5, 108.2)
- added J11: CONN_01X02, Pin_Headers:Pin_Header_Straight_1x02_Pitch2.54mm, F.Cu at (179.1, 114.3)
- added J12: CONN_01X02, Pin_Headers:Pin_Header_Straight_1x02_Pitch2.54mm, F.Cu at (168.8, 114.3)
- added J13: CONN_01X02, Pin_Headers:Pin_Header_Straight_1x02_Pitch2.54mm, F.Cu at (141.7, 114.3)
- added J14: CONN_01X02, Pin_Headers:Pin_Header_Straight_1x02_Pitch2.54mm, F.Cu at (152.4, 114.3)
- added J3: CONN_01X01, PINTST, F.Cu at (155.4, 108.2)
- added J4: CONN_01X01, PINTST, F.Cu at (153.2, 108.2)
- added J5: CONN_01X01, PINTST, F.Cu at (150.9, 108.2)
- added J6: CONN_01X01, PINTST, F.Cu at (148.6, 108.2)
- added J7: CONN_01X01, PINTST, F.Cu at (165.6, 108.2)
- added J8: CONN_01X01, PINTST, F.Cu at (167.9, 108.2)
- added J9: CONN_01X01, PINTST, F.Cu at (170.2, 108.2)
- moved C5 8.72 mm to (138.0, 108.3), turned to 0 degrees
- moved C6 1.65 mm to (185.3, 103.6)
Routing:
- net Net-(J6-Pad1): track 25.2 -> 3.99 mm
- net Net-(J5-Pad1): track 23.9 -> 3.87 mm
- net Net-(J9-Pad1): track 23.1 -> 3.90 mm
- net Net-(J7-Pad1): track 21.2 -> 3.66 mm
- net Net-(J8-Pad1): track 20.8 -> 3.78 mm
- net Net-(J4-Pad1): track 20.1 -> 3.76 mm
- net Net-(J3-Pad1): track 18.8 -> 3.64 mm
- net Net-(C1-Pad1): track 0.00 -> 5.72 mm
- net Net-(C3-Pad1): track 0.00 -> 5.67 mm
- net Net-(C5-Pad1): track 21.4 -> 25.6 mm
- net Net-(J10-Pad1): track 0.00 -> 4.01 mm
- net Net-(C2-Pad2): track 0.00 -> 3.72 mm
- net Net-(C4-Pad1): track 0.00 -> 3.59 mm
- net Net-(C6-Pad1): track 23.1 -> 19.8 mm
- added copper zone on B.Cu, net GNDA
Other:
- board outline added: 55.9 x 18.4 mm
