File: amp.sch (KiCad schematic (older format))
At the start: 16 parts, among them P1 CONN_01X05, P2 CONN_01X02, P3 CONN_01X02, P4 CONN_01X02, P5 CONN_01X02, P6 CONN_01X02, P7 CONN_01X02, U1 TDA7385

Commit message: step2
Parts:
- P4, P5, P6, P7: footprint (none) -> Connectors:bornier2
Changed lines of the file:
@@
 F 0 "P5" H 7550 2650 50  0000 C CNN
 F 1 "CONN_01X02" V 7650 2500 50  0000 C CNN
-F 2 "" H 7550 2500 50  0001 C CNN
+F 2 "Connectors:bornier2" H 7550 2500 50  0001 C CNN
 F 3 "" H 7550 2500 50  0000 C CNN
 	1    7550 2500
@@
 F 0 "P4" H 6950 2650 50  0000 C CNN
 F 1 "CONN_01X02" V 7050 2500 50  0000 C CNN
-F 2 "" H 6950 2500 50  0001 C CNN
+F 2 "Connectors:bornier2" H 6950 2500 50  0001 C CNN
 F 3 "" H 6950 2500 50  0000 C CNN
 	1    6950 2500
@@
 F 0 "P6" H 8100 2650 50  0000 C CNN
 F 1 "CONN_01X02" V 8200 2500 50  0000 C CNN
-F 2 "" H 8100 2500 50  0001 C CNN
+F 2 "Connectors:bornier2" H 8100 2500 50  0001 C CNN
 F 3 "" H 8100 2500 50  0000 C CNN
 	1    8100 2500
@@
 F 0 "P7" H 8650 2650 50  0000 C CNN
 F 1 "CONN_01X02" V 8750 2500 50  0000 C CNN
-F 2 "" H 8650 2500 50  0001 C CNN
+F 2 "Connectors:bornier2" H 8650 2500 50  0001 C CNN
 F 3 "" H 8650 2500 50  0000 C CNN
 	1    8650 2500

Commit message: final pcb for amp board
Parts:
- removed P1: CONN_01X05, symbol CONN_01X05
- removed P2, P3, P4, P5, P6, P7: CONN_01X02, Connectors:bornier2, symbol CONN_01X02
- added J1, J10, J2, J3, J4, J5, J6, J7, J8, J9: CONN_01X01, Connectors:PINTST, symbol CONN_01X01
- added J11, J12, J13, J14: CONN_01X02, Pin_Headers:Pin_Header_Straight_1x02_Pitch2.54mm, symbol CONN_01X02
Connections:
- net GNDA: now also J11.1 (P1), J12.1 (P1), J13.1 (P1), J14.1 (P1)
- net at U1.17 (OUT3+): now also J7.1 (P1)
- net at U1.19 (OUT3-): now also J8.1 (P1)
- net at U1.20 (Vcc2): now also J2.1 (P1)
- net at U1.21 (OUT4+): now also J9.1 (P1)
- net at U1.23 (OUT4-): now also J10.1 (P1)
- net at U1.3 (OUT2-): now also J6.1 (P1)
- net at U1.5 (OUT2+): now also J5.1 (P1)
- net at U1.6 (Vcc1): now also J1.1 (P1)
- net at U1.7 (OUT1-): now also J4.1 (P1)
- net at U1.9 (OUT1+): now also J3.1 (P1)
- net at C2.2: now also J12.2 (P2)
- net at C3.1: now also J13.2 (P2)
- net at C4.1: now also J14.2 (P2)
- net at C1.1: now also J11.2 (P2)
